File: Arduino.sch (KiCad schematic (older format))
At the start: 9 parts

Commit message: second "workday"
Parts:
- added SW?: SW_SPST, symbol Switch:SW_SPST
- C1, C2, C3, C4, C5: renamed from C?; symbol C -> doorhat-rescue:C
- IC1: renamed from IC?; symbol ATMEGA328P-A -> doorhat-rescue:ATMEGA328P-A
- P1: renamed from P?; symbol CONN_02X03 -> doorhat-rescue:CONN_02X03
- R13: renamed from R?; symbol R -> doorhat-rescue:R
- Y1: renamed from Y?; symbol Crystal -> doorhat-rescue:Crystal
Connections:
- net labels added: cardreader_clk, cardreader_data, clk, mfr_rfid_nrstpd, mfr_rfid_ss, miso, mosi, sck, serial_program, serial_rfid_data, serial_rfid_enable, xtal1, xtal2
- net labels removed: avr_clk, avr_miso, avr_mosi
- wire segments 45 -> 61
Other:
- moved on the sheet: C1, C4, C5, R13, Y1
