File: doorhat.sch (KiCad schematic (older format))
At the start: 26 parts

Commit message: second "workday"
Parts:
- removed D? (x5): LED, symbol LED
- removed Q?: BC547, TO_SOT_Packages_THT:TO-92_Molded_Narrow, symbol BC547
- removed R? (x4): R_Small, symbol R_Small
- added J? (x8): Conn_01x02, symbol Connector_Generic:Conn_01x02
- added J?: Conn_01x06, symbol Connector_Generic:Conn_01x06
- added J?: Conn_01x07, symbol Connector_Generic:Conn_01x07
- added J?: Conn_01x04, symbol Connector_Generic:Conn_01x04
- added Q?: IRLZ44N, Package_TO_SOT_THT:TO-220-3_Vertical, symbol Transistor_FET:IRLZ44N
- added Q?: BC547, TO_SOT_Packages_THT:TO-92_Molded_Narrow, symbol doorhat-rescue:BC547
- added R?: R_Small, Resistors_SMD:R_0805_HandSoldering, symbol doorhat-rescue:R_Small
- added R? (x5): 10k, Resistors_SMD:R_0805_HandSoldering, symbol doorhat-rescue:R_Small
- added R?: 1k, Resistors_SMD:R_0805_HandSoldering, symbol doorhat-rescue:R_Small
- added RLY?: EC2-5NU, digikey-footprints:Relay_THT_EC2, symbol dk_Signal-Relays-Up-to-2-Amps:EC2-5NU
- added U?: TXB0104PWR, digikey-footprints:TSSOP-14_W4.4mm, symbol dk_Logic-Translators-Level-Shifters:TXB0104PWR
- CONN1: renamed from CONN?; symbol RaspberryPi_40W_GPIO_Connector -> doorhat-rescue:RaspberryPi_40W_GPIO_Connector
- Q1, Q2, Q4, Q5, Q6: renamed from Q?; symbol BC547 -> doorhat-rescue:BC547
- R10, R11, R12, R4, R5, R6, R7, R9: renamed from R?; footprint (none) -> Resistors_SMD:R_0805_HandSoldering; symbol R_Small -> doorhat-rescue:R_Small
- SP1: renamed from SP?; symbol SPEAKER -> doorhat-rescue:SPEAKER
- U1: renamed from U?; symbol L6234 -> doorhat-rescue:L6234
Connections:
- net labels added: +12V, Daymode_button, buzzer_lock, cardreader_clk, cardreader_data, cardreader_led_green, cardreader_led_green_control, cardreader_led_yellow, cardreader_led_yellow_control, daymode_led_+, daymode_led_-, door_direction, door_enable, door_lock_button, door_sens_1, door_sens_2, led_daymode, led_lock, lock_led_+, lock_led_-, mfr_rfid_nrstpd, mfr_rfid_ss, miso, mosi, sck, serial_hash, serial_program, serial_rfid_data, serial_rfid_enable
- net labels removed: ld_green
- wire segments 56 -> 105
Other:
- note added: "- RC-led i serie med gaten på mosfetten,\nsådan at trækspolen ikke kan brændes af ved computerfejl"
- note added: "Ting der skal testes/måles på døren fysisk:"
- note added: "Ting i koden:"
- note added: "door connectors\n"
- note added: "door lock next time..... håndtering\n"
- note added: "hvordan forsynes led'erne på kortlæseren"
- note added: "inside door open button"
- note added: "noter til fremtidige revisioner:"
- note added: "relæ hvile stilling skal være åben polaritet"
- note removed: "[Cardreader\nred LED???]"
- moved on the sheet: CONN1, Q1, Q2, Q4, Q5, Q6, R10, R11, R12, R4, R5, R6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
